Commit message: Dépôt final du projet : Simulation + Code + Guide README

File: install/mobile_robot/share/mobile_robot/model/robot.xacro (robot description, xacro)
@@ -1 +1,113 @@
-/home/user/ws_mobile_robot/build/mobile_robot/model/robot.xacro
+<?xml version="1.0"?>
+<robot xmlns:xacro="http://www.ros.org/wiki/xacro" name="robot">
+    <xacro:include filename="robot.gazebo" />
+    <xacro:property name="base_length" value="0.6"/>
+    <xacro:property name="base_width" value="0.4"/>
+    <xacro:property name="base_height" value="0.2"/>
+    <xacro:property name="wheel_radius" value="0.1"/>
+    <xacro:property name="wheel_width" value="0.05"/>
+    <xacro:property name="wheel_ygap" value="0.05"/>
+    <xacro:property name="wheel_zoff" value="0.05"/>
+    <xacro:property name="wheel_xoff" value="0.12"/>
+    <material name="blue"><color rgba="0 0 1 1"/></material>
+    <material name="black"><color rgba="0 0 0 1"/></material>
+    <xacro:macro name="box_inertia" params="m w h d">
+        <inertial>
+            <origin xyz="0 0 0" rpy="${pi/2} 0 ${pi/2}"/>
+            <mass value="${m}"/>
+            <inertia ixx="${(m/12) * (h*h + d*d)}" ixy="0.0" ixz="0.0" iyy="${(m/12) * (w*w + d*d)}" iyz="0.0" izz="${(m/12) * (w*w + h*h)}"/>
+        </inertial>
+    </xacro:macro>
+    <xacro:macro name="cylinder_inertia" params="m r h">
+        <inertial>
+            <origin xyz="0 0 0" rpy="${pi/2} 0 0" />
+            <mass value="${m}"/>
+            <inertia ixx="${(m/12) * (3*r*r + h*h)}" ixy="0" ixz="0" iyy="${(m/12) * (3*r*r + h*h)}" iyz="0" izz="${(m/2) * (r*r)}"/>
+        </inertial>
+    </xacro:macro>
+    <link name="base_footprint"/>
+    <joint name="base_joint" type="fixed">
+        <parent link="base_footprint"/>
+        <child link="base_link"/>
+        <origin xyz="0 0 ${wheel_radius + wheel_zoff}" rpy="0 0 0"/>
+    </joint>
+    <link name="base_link">
+        <visual>
+            <geometry><box size="${base_length} ${base_width} ${base_height}"/></geometry>
+            <material name="blue"/>
+        </visual>
+        <collision>
+            <geometry><box size="${base_length} ${base_width} ${base_height}"/></geometry>
+        </collision>
+        <xacro:box_inertia m="15" w="${base_width}" h="${base_height}" d="${base_length}"/>
+    </link>
+    <xacro:macro name="wheel" params="prefix x_reflect y_reflect">
+        <link name="${prefix}_link">
+            <visual>
+                <origin xyz="0 0 0" rpy="${pi/2} 0 0"/>
+                <geometry><cylinder radius="${wheel_radius}" length="${wheel_width}"/></geometry>
+                <material name="black"/>
+            </visual>
+            <collision>
+                <origin xyz="0 0 0" rpy="${pi/2} 0 0"/>
+                <geometry><cylinder radius="${wheel_radius}" length="${wheel_width}"/></geometry>
+            </collision>
+            <xacro:cylinder_inertia m="0.5" r="${wheel_radius}" h="${wheel_width}"/>
+        </link>
+        <joint name="${prefix}_joint" type="continuous">
+            <parent link="base_link"/>
+            <child link="${prefix}_link"/>
+            <origin xyz="${x_reflect*wheel_xoff} ${y_reflect*(base_width/2+wheel_ygap)} ${-wheel_zoff}" rpy="0 0 0"/>
+            <axis xyz="0 1 0"/>
+        </joint>
+    </xacro:macro>
+    <xacro:wheel prefix="drivewhl_l" x_reflect="-1" y_reflect="1"/>
+    <xacro:wheel prefix="drivewhl_r" x_reflect="-1" y_reflect="-1"/>
+    <link name="caster_wheel">
+        <visual>
+            <geometry><sphere radius="0.05"/></geometry>
+            <material name="black"/>
+        </visual>
+        <collision>
+            <geometry><sphere radius="0.05"/></geometry>
+        </collision>
+        <xacro:cylinder_inertia m="0.1" r="0.05" h="0.05"/>
+    </link>
+    <joint name="caster_wheel_joint" type="fixed">
+        <parent link="base_link"/>
+        <child link="caster_wheel"/>
+        <origin xyz="0.2 0 -0.05" rpy="0 0 0"/>
+    </joint>
+    <!-- LIDAR -->
+    <link name="laser_frame">
+        <visual>
+            <geometry><cylinder radius="0.05" length="0.04"/></geometry>
+            <material name="black"/>
+        </visual>
+        <collision>
+            <geometry><cylinder radius="0.05" length="0.04"/></geometry>
+        </collision>
+        <xacro:cylinder_inertia m="0.1" r="0.05" h="0.04"/>
+    </link>
+    <joint name="laser_joint" type="fixed">
+        <parent link="base_link"/>
+        <child link="laser_frame"/>
+        <origin xyz="0.1 0 0.12" rpy="0 0 0"/>
+    </joint>
+    <!-- CAMERA -->
+    <link name="camera_link">
+        <visual>
+            <geometry><box size="0.05 0.05 0.05"/></geometry>
+            <material name="black"/>
+        </visual>
+        <collision>
+            <geometry><box size="0.05 0.05 0.05"/></geometry>
+        </collision>
+        <xacro:box_inertia m="0.1" w="0.05" h="0.05" d="0.05"/>
+    </link>
+    <joint name="camera_joint" type="fixed">
+        <parent link="base_link"/>
+        <child link="camera_link"/>
+        <origin xyz="0.28 0 0.05" rpy="0 0 0"/>
+    </joint>
+</robot>

File: src/mobile_robot/model/robot.xacro (robot description, xacro)
@@ -79,4 +79,5 @@
         <origin xyz="0.2 0 -0.05" rpy="0 0 0"/>
     </joint>
+    <!-- LIDAR -->
     <link name="laser_frame">
         <visual>
@@ -94,28 +95,19 @@
         <origin xyz="0.1 0 0.12" rpy="0 0 0"/>
     </joint>
-    <gazebo reference="laser_frame">
-        <sensor name="lidar" type="gpu_ray">
-            <pose> 0 0 0 0 0 0 </pose>
-            <visualize>true</visualize>
-            <update_rate>10</update_rate>
-            <ray>
-                <scan>
-                    <horizontal>
-                        <samples>360</samples>
-                        <min_angle>-3.14</min_angle>
-                        <max_angle>3.14</max_angle>
-                    </horizontal>
-                </scan>
-                <range>
-                    <min>0.3</min>
-                    <max>12</max>
-                </range>
-            </ray>
-            <plugin filename="gz-sim-sensors-system" name="gz::sim::systems::Sensors">
-                <render_engine>ogre2</render_engine>
-            </plugin>
-            <topic>scan</topic>
-            <gz_frame_id>laser_frame</gz_frame_id>
-        </sensor>
-    </gazebo>
+    <!-- CAMERA -->
+    <link name="camera_link">
+        <visual>
+            <geometry><box size="0.05 0.05 0.05"/></geometry>
+            <material name="black"/>
+        </visual>
+        <collision>
+            <geometry><box size="0.05 0.05 0.05"/></geometry>
+        </collision>
+        <xacro:box_inertia m="0.1" w="0.05" h="0.05" d="0.05"/>
+    </link>
+    <joint name="camera_joint" type="fixed">
+        <parent link="base_link"/>
+        <child link="camera_link"/>
+        <origin xyz="0.28 0 0.05" rpy="0 0 0"/>
+    </joint>
 </robot>
